File: FlameSensorSender/KiCAD/FlameSensorSender/FlameSensorSender.kicad_pcb (KiCad board)
At the start: 2 copper layers, 80 x 40 mm, 23 parts, among them J1 SWD, J2 Sharp GP2Y1014AUOF, Q1 AO3400A, Q2 AO3400A, U1 STM32F103C6Tx, U2 Ai-Thinker-Ra-02, U3 MT3608 module

Commit message: dev
Parts:
- added C12: 22u, Capacitor_SMD:C_0603_1608Metric_Pad1.08x0.95mm_HandSolder, F.Cu at (118.4, 99.4)
- added C5: 105, 0603, Capacitor_SMD:C_0603_1608Metric_Pad1.08x0.95mm_HandSolder, B.Cu at (75.4, 80.5)
- added C7: 22u, Capacitor_SMD:C_0603_1608Metric_Pad1.08x0.95mm_HandSolder, F.Cu at (89.6, 69.5)
- added C8: 22u, Capacitor_SMD:C_0603_1608Metric_Pad1.08x0.95mm_HandSolder, F.Cu at (93.6, 61.5)
- added C9: 22u, Capacitor_SMD:C_0603_1608Metric_Pad1.08x0.95mm_HandSolder, F.Cu at (114.1, 106.9)
- added L1: 470n, Inductor_SMD:L_Coilcraft_XxL4020, F.Cu at (83.4, 66.7)
- added L2: 470n, Inductor_SMD:L_Coilcraft_XxL4020, F.Cu at (84.4, 32.3)
- added R1: 10k, 0603, Resistor_SMD:R_0603_1608Metric_Pad0.98x0.95mm_HandSolder, B.Cu at (75.4, 75.4)
- added R11: 100k Rpg, Resistor_SMD:R_0603_1608Metric_Pad0.98x0.95mm_HandSolder, F.Cu at (122.8, 101.9)
- added R12: 806k Rfbt, Resistor_SMD:R_0603_1608Metric_Pad0.98x0.95mm_HandSolder, F.Cu at (122.8, 104.4)
- added R13: 91k Rfbb, Resistor_SMD:R_0603_1608Metric_Pad0.98x0.95mm_HandSolder, F.Cu at (122.8, 106.9)
- added R4: 100k Rpg, Resistor_SMD:R_0603_1608Metric_Pad0.98x0.95mm_HandSolder, F.Cu at (93.4, 65.5)
- added R5: 511k Rfbt, Resistor_SMD:R_0603_1608Metric_Pad0.98x0.95mm_HandSolder, F.Cu at (94.4, 68.4)
- added R6: 91k Rfbb, Resistor_SMD:R_0603_1608Metric_Pad0.98x0.95mm_HandSolder, F.Cu at (92.4, 68.4)
- added SW1: SW_Push, Button_Switch_THT:SW_PUSH_6mm_H4.3mm, B.Cu at (66.4, 74.5)
- added U4: TPS63802DLAR, Footprints:VREG_TPS63802DLAR, F.Cu at (118.8, 119.0)
- U3: value MT3608 module -> TPS63802DLAR; footprint Footprints:MT3608_module_SMT -> Footprints:VREG_TPS63802DLAR
- moved BT1 54.9 mm to (84.4, 71.5), turned to 0 degrees
- moved R3 29.2 mm to (138.4, 78.5), turned to 180 degrees
- moved Q1 24.3 mm to (138.4, 73.6), turned to 180 degrees
- moved D1 20.8 mm to (138.4, 68.5), turned to 0 degrees
- moved R2 19.3 mm to (138.4, 64.5), turned to 0 degrees
- moved C3 12.9 mm to (116.5, 76.5), turned to 90 degrees
- moved C6 12.2 mm to (113.5, 51.5), turned to -90 degrees
- moved U3 8.18 mm to (89.4, 66.5), turned to 180 degrees
- moved C11 7.08 mm to (75.5, 67.5), turned to 180 degrees
- moved C2 5.04 mm to (100.3, 69.5)
- moved D2 5.04 mm to (98.3, 50.5)
- moved Q2 5.04 mm to (102.4, 49.5)
- moved R7 5.04 mm to (103.3, 54.5)
- moved R8 5.04 mm to (101.3, 76.5)
- moved R9 5.04 mm to (101.3, 73.5)
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- renumbered C7 to C10, C6 to C11, C5 to C6, J2 to J1, J1 to J2, R6 to R10, R1 to R2, R2 to R3, R3 to R7, R4 to R8, R5 to R9
Connections:
- net /VDD LORA renamed Net-(D1-K)
- BT1 pad 1: +3V3 -> /BATTERY_IN
- C1 pad 1: +3V3 -> /+3V3 regulated
- C11 pad 2: +3V3 -> /+3V3 regulated
- C2 pad 1: +3V3 -> /+3V3 regulated
- C3 pad 1: +3V3 -> /+3V3 regulated
- C4 pad 1: +3V3 -> /+3V3 regulated
- C6 pad 1: +3V3 -> /+3V3 regulated
- J1 pad 6: /+5V0 -> Net-(D2-K)
- J2 pad 1: +3V3 -> /+3V3 regulated
- Q1 pad 2: +3V3 -> /+3V3 regulated
- Q2 pad 2: +3V3 -> /+5V0 regulated
- R10 pad 2: /+5V0 -> Net-(D2-K)
- R2 pad 2: +3V3 -> /+3V3 regulated
- U1 pad 1: +3V3 -> /+3V3 regulated
- U1 pad 24: +3V3 -> /+3V3 regulated
- U1 pad 36: +3V3 -> /+3V3 regulated
- U1 pad 48: +3V3 -> /+3V3 regulated
- U1 pad 7: unconnected-(U1-NRST-Pad7) -> /RESET_PIN
- U1 pad 8: VSSA -> GNDD
- U1 pad 9: +3V3 -> /+3V3 regulated
- U3 pad 1: Net-(D2-K) -> /BATTERY_IN
- U3 pad 4: /+5V0 -> Net-(U3-FB)
Routing:
- net /SWCLK: track 47.1 -> 0.00 mm, vias 1 -> 0
- net /SWDIO: track 42.2 -> 0.00 mm, vias 3 -> 0
- net +3V3: track 41.8 -> 0.00 mm, vias 3 -> 0
- net Net-(J1-Pin_5): track 35.1 -> 0.00 mm, vias 2 -> 0
- net Net-(U1-PA5): track 33.9 -> 0.00 mm, vias 2 -> 0
- net /+3V3 regulated: track 0.00 -> 32.4 mm
- net Net-(D2-K): track 32.2 -> 0.00 mm
- net Net-(U1-PA6): track 31.8 -> 0.00 mm, vias 2 -> 0
- net /PB12: track 31.8 -> 0.00 mm, vias 2 -> 0
- net /PB0: track 30.2 -> 0.00 mm
- net Net-(U1-PA7): track 29.7 -> 0.00 mm
- net Net-(U1-PA4): track 24.6 -> 0.00 mm
- net /LORA EN: track 22.3 -> 0.00 mm, vias 2 -> 0
- net /+5V0: track 19.4 -> 0.00 mm, vias 1 -> 0
- net /SENSOR DATA: track 19.2 -> 0.00 mm, vias 2 -> 0
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- added copper zone on F.Cu, net /+3V3 regulated
- removed copper zone on F.Cu, net +3V3

Commit message: dev
Parts:
- BT1: value CR123A 3V -> AA 2pcs 3V0-3V6 at start
Changed lines of the file:
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@@
 			)
 		)
-		(property "Value" "CR123A 3V"
+		(property "Value" "AA 2pcs 3V0-3V6 at start"
 			(at 29.165 -8.715 0)
 			(layer "B.Fab")
