File: KiCAD/FlameSensorSender/FlameSensorSender.kicad_pcb (KiCad board)
At the start: 2 copper layers, 80 x 40 mm, 39 parts, among them J1 Sharp GP2Y1014AUOF, J2 SWD, Q1 AO3400A, Q2 AO3400A, SW1 SW_Push, U1 STM32F103C6Tx, U2 Ai-Thinker-Ra-02, U3 TPS63802DLAR, U4 TPS63802DLAR

Commit message: dev
Parts:
- removed the C7 at (89.6, 69.5)
- removed the C8 at (93.6, 61.5)
- removed the R5 at (94.4, 68.4)
- removed the R6 at (92.4, 68.4)
- removed the R7 at (103.3, 54.5)
- added C10: 470u, Capacitor_SMD:C_0805_2012Metric_Pad1.18x1.45mm_HandSolder, B.Cu at (73.4, 80.5)
- added C11: 22u, Capacitor_SMD:C_0603_1608Metric_Pad1.08x0.95mm_HandSolder, F.Cu at (87.4, 80.4)
- added C13: 22u, Capacitor_SMD:C_0603_1608Metric_Pad1.08x0.95mm_HandSolder, F.Cu at (80.6, 102.1)
- added J3: USB_C_Receptacle_PowerOnly_6P, Connector_USB:USB_C_Receptacle_GCT_USB4135-GF-A_6P_TopMnt_Horizontal, B.Cu at (66.4, 74.5)
- added R10: 91k Rfbb, Resistor_SMD:R_0603_1608Metric_Pad0.98x0.95mm_HandSolder, F.Cu at (78.4, 82.5)
- added R14: 470k,0603, Resistor_SMD:R_0201_0603Metric_Pad0.64x0.40mm_HandSolder, F.Cu at (92.8, 113.5)
- added R15: 100k Rpg, Resistor_SMD:R_0603_1608Metric_Pad0.98x0.95mm_HandSolder, F.Cu at (80.6, 112.1)
- added R16: 806k Rfbt, Resistor_SMD:R_0603_1608Metric_Pad0.98x0.95mm_HandSolder, F.Cu at (80.6, 114.6)
- added R17: 91k Rfbb, Resistor_SMD:R_0603_1608Metric_Pad0.98x0.95mm_HandSolder, F.Cu at (63.3, 115.5)
- added R8: 100k Rpg, Resistor_SMD:R_0603_1608Metric_Pad0.98x0.95mm_HandSolder, F.Cu at (83.4, 80.4)
- added R9: 511k Rfbt, Resistor_SMD:R_0603_1608Metric_Pad0.98x0.95mm_HandSolder, F.Cu at (85.4, 80.4)
- BT1: value AA 2pcs 3V0-3V6 at start -> AA 2pcs
- C1, C2, C3, C6: footprint Capacitor_SMD:C_0805_2012Metric_Pad1.18x1.45mm_HandSolder -> Capacitor_SMD:C_0603_1608Metric_Pad1.08x0.95mm_HandSolder
- C5: renamed from C4; footprint Capacitor_SMD:C_0805_2012Metric_Pad1.18x1.45mm_HandSolder -> Capacitor_SMD:C_0603_1608Metric_Pad1.08x0.95mm_HandSolder
- C7: renamed from C11; footprint Capacitor_SMD:C_0805_2012Metric_Pad1.18x1.45mm_HandSolder -> Capacitor_SMD:C_0603_1608Metric_Pad1.08x0.95mm_HandSolder
- C8: renamed from C10; footprint Capacitor_SMD:C_0805_2012Metric_Pad1.18x1.45mm_HandSolder -> Capacitor_SMD:C_0603_1608Metric_Pad1.08x0.95mm_HandSolder
- D1, D2: value 1N5819 -> SS34; footprint Diode_SMD:D_0805_2012Metric_Pad1.15x1.40mm_HandSolder -> Diode_SMD:D_SMA; moved to B.Cu
- Q1, Q2: value AO3400A -> AO3401A; footprint Package_TO_SOT_SMD:SOT-23 -> Package_TO_SOT_SMD:SOT-23_Handsoldering
- R11: value 100k Rpg -> 5.1k; footprint Resistor_SMD:R_0603_1608Metric_Pad0.98x0.95mm_HandSolder -> Resistor_SMD:R_0201_0603Metric_Pad0.64x0.40mm_HandSolder
- R12: value 806k Rfbt -> 5.1k; footprint Resistor_SMD:R_0603_1608Metric_Pad0.98x0.95mm_HandSolder -> Resistor_SMD:R_0201_0603Metric_Pad0.64x0.40mm_HandSolder
- R13: value 91k Rfbb -> 1k,0603; footprint Resistor_SMD:R_0603_1608Metric_Pad0.98x0.95mm_HandSolder -> Resistor_SMD:R_0201_0603Metric
- R2: footprint Resistor_SMD:R_0805_2012Metric_Pad1.20x1.40mm_HandSolder -> Resistor_SMD:R_0201_0603Metric_Pad0.64x0.40mm_HandSolder
- R3: value 10k -> 1k,0603; footprint Resistor_SMD:R_0805_2012Metric_Pad1.20x1.40mm_HandSolder -> Resistor_SMD:R_0201_0603Metric_Pad0.64x0.40mm_HandSolder
- R4: value 100k Rpg -> 470k,0603; footprint Resistor_SMD:R_0603_1608Metric_Pad0.98x0.95mm_HandSolder -> Resistor_SMD:R_0201_0603Metric_Pad0.64x0.40mm_HandSolder
- R5: renamed from R8; footprint Resistor_SMD:R_0805_2012Metric_Pad1.20x1.40mm_HandSolder -> Resistor_SMD:R_0603_1608Metric_Pad0.98x0.95mm_HandSolder
- R6: renamed from R9; footprint Resistor_SMD:R_0805_2012Metric_Pad1.20x1.40mm_HandSolder -> Resistor_SMD:R_0603_1608Metric_Pad0.98x0.95mm_HandSolder
- R7: renamed from R10; footprint Resistor_SMD:R_0805_2012Metric_Pad1.20x1.40mm_HandSolder -> Resistor_SMD:R_0603_1608Metric_Pad0.98x0.95mm_HandSolder
- moved L2 69.4 mm to (85.6, 101.7), turned to 0 degrees
- moved R11 63.3 mm to (66.4, 73.1), turned to 90 degrees
- moved R12 63.1 mm to (66.4, 76.1), turned to -90 degrees
- moved R4 62.3 mm to (62.6, 119.6), turned to 0 degrees
- moved D1 60.2 mm to (78.4, 73.5), turned to 90 degrees
- moved Q2 50.9 mm to (99.7, 100.4), turned to 0 degrees
- moved C9 47.0 mm to (77.4, 77.5), turned to 90 degrees
- moved C12 37.8 mm to (80.6, 99.6)
- moved D2 33.2 mm to (74.4, 73.5)
- moved U4 28.0 mm to (103.3, 95.6)
- moved C3 24.2 mm to (135.4, 91.5), turned to 0 degrees
- moved R3 24.1 mm to (114.4, 76.5), turned to 90 degrees
- moved R13 22.5 mm to (100.5, 103.5)
- moved C6 22.3 mm to (93.0, 60.5), turned to 180 degrees
- moved R7 21.8 mm to (55.4, 44.4)
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- renumbered C5 to C4, J2 to J1, J1 to J2
Connections:
- BT1 pad 1: /BATTERY_IN -> Net-(BT1-+)
- C1 pad 1: /+3V3 regulated -> +3V3
- C12 pad 1: /+5V0 regulated -> Net-(Q2-D)
- C2 pad 1: /+3V3 regulated -> +3V3
- C3 pad 1: /+3V3 regulated -> +3V3
- C5 pad 1: /+3V3 regulated -> +3V3
- C6 pad 1: /+3V3 regulated -> +3V3
- C7 pad 2: /+3V3 regulated -> +3V3
- C9 pad 1: /BATTERY_IN -> VRAW
- D1 pad 1: Net-(D1-K) -> VRAW
- D1 pad 2: Net-(D1-A) -> Net-(BT1-+)
- D2 pad 1: Net-(D2-K) -> VRAW
- J1 pad 1: /+3V3 regulated -> +3V3
- J2 pad 6: Net-(D2-K) -> +5V0
- Q1 pad 2: /+3V3 regulated -> +3V3
- Q1 pad 3: Net-(D1-A) -> Net-(Q1-D)
- Q2 pad 2: /+5V0 regulated -> VRAW
- Q2 pad 3: Net-(D2-A) -> Net-(Q2-D)
- R1 pad 1: /+3V3 regulated -> +3V3
- R11 pad 1: /+5V0 regulated -> Net-(J3-CC2)
- R11 pad 2: Net-(U4-PG) -> GNDD
- R12 pad 1: /+5V0 regulated -> Net-(J3-CC1)
- R12 pad 2: Net-(U4-FB) -> GNDD
- R13 pad 1: Net-(U4-FB) -> Net-(Q2-G)
- R13 pad 2: GNDD -> SENSOR EN
- R2 pad 2: /+3V3 regulated -> +3V3
- R3 pad 1: Net-(Q1-G) -> /LORA EN
- R3 pad 2: /LORA EN -> Net-(Q1-G)
- R4 pad 1: /+3V3 regulated -> Net-(Q1-G)
- R4 pad 2: Net-(U3-PG) -> +3V3
- R7 pad 2: Net-(D2-K) -> +5V0
- U1 pad 1: /+3V3 regulated -> +3V3
- U1 pad 21: /SENSOR EN -> SENSOR EN
- U1 pad 24: /+3V3 regulated -> +3V3
- U1 pad 36: /+3V3 regulated -> +3V3
- U1 pad 48: /+3V3 regulated -> +3V3
- U1 pad 9: /+3V3 regulated -> +3V3
- U2 pad 3: Net-(D1-K) -> Net-(Q1-D)
- U3 pad 1: /BATTERY_IN -> VRAW
- U3 pad 10: /BATTERY_IN -> VRAW
- U3 pad 6: /+3V3 regulated -> +3V3
- U4 pad 1: /BATTERY_IN -> Net-(Q2-D)
- U4 pad 10: /BATTERY_IN -> Net-(Q2-D)
- U4 pad 6: /+5V0 regulated -> +5V0
Routing:
- net Net-(U1-PA6): track 0.00 -> 37.9 mm, vias 0 -> 2
- net Net-(U1-PA5): track 0.00 -> 37.8 mm
- net Net-(U1-PA7): track 0.00 -> 37.5 mm, vias 0 -> 2
- net +3V3: track 0.00 -> 34.3 mm
- net /+3V3 regulated: track 32.4 -> 0.00 mm
- net Net-(U1-PA4): track 0.00 -> 30.5 mm
- net VRAW: track 0.00 -> 17.8 mm, vias 0 -> 1
- net /BATTERY_IN: track 9.57 -> 0.00 mm
- net Net-(D1-A): track 5.89 -> 0.00 mm
- net Net-(BT1-+): track 0.00 -> 5.83 mm
- net Net-(D1-K): track 5.83 -> 0.00 mm
- net Net-(D2-A): track 0.00 -> 5.58 mm
- net Net-(U2-~{RESET}): track 5.00 -> 0.00 mm
- net Net-(U3-FB): track 5.48 -> 8.99 mm
- net Net-(J3-CC1): track 0.00 -> 3.31 mm, vias 0 -> 1
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- removed copper zone on F.Cu, net /+3V3 regulated
