File: KiCAD/FlameSensorSender/FlameSensorSender.kicad_pcb (KiCad board)
At the start: 2 copper layers, 80 x 40 mm, 49 parts, among them J1 SWD, J3 JST-PH B2B-PH-K-S, J5 JST-PH B2B-PH-K-S, J6 Sharp GP2Y1014AUOF, J7 USB_C_Receptacle_PowerOnly_6P, Q1 AO3401A, Q2 AO3401A, SW1 SW_Push, U1 STM32F103C6Tx, U2 Ai-Thinker-Ra-02, U3 TPS63802DLAR, U4 TPS63802DLAR

Commit message: dev
Other:
- board text added: "Dust Sensor"
- board text added: "LED"
Changed lines of the file:
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@@
 		(tags "connector JST PH vertical")
 		(property "Reference" "J3"
-			(at 1 2.9 0)
+			(at -2.370062 2.860412 0)
 			(layer "B.SilkS")
 			(effects
@@
 		)
 	)
+	(gr_text "LED"
+		(at 63.813369 60.850064 180)
+		(layer "B.SilkS" knockout)
+		(effects
+			(font
+				(size 1 1)
+				(thickness 0.1)
+			)
+			(justify left bottom mirror)
+		)
+	)
 	(gr_text "SWDIO"
 		(at 75.479665 44.684327 180)
 		(layer "B.SilkS" knockout)
 		(effects
+			(font
+				(size 1 1)
+				(thickness 0.1)
+			)
+			(justify left bottom mirror)
+		)
+	)
+	(gr_text "Dust Sensor"
+		(at 65.4175 48.5 90)
+		(layer "B.SilkS" knockout)
+		(effects

Commit message: dev
Parts:
- added BZ1: Buzzer, Buzzer_Beeper:Buzzer_12x9.5RM7.6, F.Cu at (104.6, 95.5)
- added Q1: AO3400A, Package_TO_SOT_SMD:SOT-23, F.Cu at (111.9, 106.6)
- added R3: 1k,0603, Resistor_SMD:R_0603_1608Metric_Pad0.98x0.95mm_HandSolder, F.Cu at (116.5, 105.5)
- renumbered Q1 to Q2, Q2 to Q3, R9 to R10, R10 to R11, R11 to R12, R12 to R13, R13 to R14, R14 to R15, R15 to R16, R16 to R17, R17 to R18, R18 to R19, R19 to R20, R3 to R6, R6 to R9

Commit message: dev
Parts:
- removed BZ1: Buzzer, Buzzer_Beeper:Buzzer_12x9.5RM7.6
- C8: moved to B.Cu
- J3, J6: moved to F.Cu
- Q3: value AO3401A -> AO3400A; footprint Package_TO_SOT_SMD:SOT-23-3 -> Package_TO_SOT_SMD:SOT-23
- R5: renamed from R6; moved to B.Cu
- R8: renamed from R10; moved to B.Cu
- R9: value 110,0603 -> 330,0603
- moved Q2 26.0 mm to (105.4, 81.4), turned to -90 degrees
- moved R10 25.7 mm to (110.4, 80.5), turned to 90 degrees
- moved R8 6.24 mm to (64.4, 49.5)
- moved C8 2.28 mm to (64.4, 57.6), turned to -90 degrees
- moved R5 2.09 mm to (64.4, 62.6)
- moved J5 2.00 mm to (93.4, 81.5), turned to 0 degrees
- moved J6 1.83 mm to (67.4, 58.5)
- moved J3 1.00 mm to (68.4, 65.5)
- turned R20 to -90 degrees
- renumbered Q2 to Q1, Q1 to Q2, R3 to R10, R4 to R3, R5 to R4, R7 to R6, R8 to R7
Connections:
- C12 pad 1: Net-(Q3-D) -> VRAW
- C12 pad 2: GNDD -> Net-(Q3-D)
- C13 pad 2: GNDD -> Net-(Q3-D)
- J5 pad 1: Net-(J5-Pin_1) -> VRAW
- J5 pad 2: GNDD -> Net-(J5-Pin_2)
- Q2 pad 1: Net-(Q1-G) (its old number) -> Net-(Q2-G)
- Q2 pad 3: Net-(BZ1--) -> Net-(Q2-D)
- Q3 pad 2: VRAW -> GNDD
- R10 pad 1: unconnected-(R3-Pad1) -> Net-(Q2-G)
- R10 pad 2: Net-(Q1-G) (its old number) -> /INFO_BUZZER
- R17 pad 2: VRAW -> GNDD
- R20 pad 2: GNDD -> Net-(Q3-D)
- R9 pad 1: /INFO_BUZZER -> Net-(Q2-D)
- R9 pad 2: Net-(J5-Pin_1) -> Net-(J5-Pin_2)
- U4 pad 1: Net-(Q3-D) -> VRAW
- U4 pad 10: Net-(Q3-D) -> VRAW
- U4 pad 2: GNDD -> Net-(Q3-D)
- U4 pad 3: GNDD -> Net-(Q3-D)
- U4 pad 8: GNDD -> Net-(Q3-D)
Routing:
- net Net-(Q3-D): track 8.59 -> 31.1 mm, vias 0 -> 2
- net Net-(Q2-D): track 0.00 -> 5.69 mm
- net Net-(J5-Pin_2): track 0.00 -> 5.38 mm
- net Net-(J5-Pin_1): track 5.38 -> 0.00 mm
- net +5V0: track 36.5 -> 31.3 mm
- net /INFO_BUZZER: track 14.0 -> 19.1 mm
- net GNDD: track 65.7 -> 61.0 mm
- net Net-(Q2-G): track 0.00 -> 4.48 mm
- net VRAW: track 74.0 -> 77.2 mm, vias 2 -> 4
- net Net-(J6-Pin_5): track 34.0 -> 35.8 mm
- net Net-(U4-FB): track 15.6 -> 16.7 mm
- net /INFO_LED: track 33.5 -> 32.6 mm, vias 2 -> 3
- net Net-(J6-Pin_1): track 10.8 -> 10.1 mm, vias 0 -> 2
- net /PB12: track 33.9 -> 34.6 mm
Other:
- board size 80 x 40 mm -> 80 x 42 mm

Commit message: dev
Connections:
- C12 pad 2: Net-(Q3-D) -> GNDD2
- C13 pad 2: Net-(Q3-D) -> GNDD2
- Q2 pad 2: GNDD -> GNDD2
- Q3 pad 3: Net-(Q3-D) -> GNDD2
- R20 pad 2: Net-(Q3-D) -> GNDD2
- U4 pad 2: Net-(Q3-D) -> GNDD2
- U4 pad 3: Net-(Q3-D) -> GNDD2
- U4 pad 8: Net-(Q3-D) -> GNDD2
Routing:
- net GNDD2: track 0.00 -> 61.5 mm, vias 0 -> 3
- net Net-(Q3-D): track 31.1 -> 0.00 mm, vias 2 -> 0
- net GNDD: track 61.0 -> 58.6 mm, vias 38 -> 37
Changed lines of the file:
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@@
 	(net 68 "/INFO_BUZZER")
 	(net 69 "unconnected-(U1-PB14-Pad27)")
-	(net 70 "Net-(Q3-D)")
+	(net 70 "GNDD2")
 	(net 71 "Net-(Q3-G)")
 	(footprint "Resistor_SMD:R_0603_1608Metric_Pad0.98x0.95mm_HandSolder"
@@
 			(layers "F.Cu" "F.Mask" "F.Paste")
 			(roundrect_rratio 0.25)
-			(net 70 "Net-(Q3-D)")
+			(net 70 "GNDD2")
 			(pinfunction "D")
 			(pintype "passive")
@@
 			(layers "F.Cu" "F.Paste")
 			(roundrect_rratio 0.2)
-			(net 70 "Net-(Q3-D)")
+			(net 70 "GNDD2")
 			(pinfunction "MODE")
 			(pintype "input")
@@
 			(layers "F.Cu" "F.Paste")
 			(roundrect_rratio 0.2)
-			(net 70 "Net-(Q3-D)")
+			(net 70 "GNDD2")
 			(pinfunction "AGND")
 			(pintype "power_in")
@@
 			(layers "F.Cu")
 			(roundrect_rratio 0.2)
-			(net 70 "Net-(Q3-D)")
+			(net 70 "GNDD2")
 			(pinfunction "GND")
 			(pintype "power_in")
@@
 			(layers "F.Cu" "F.Mask" "F.Paste")
 			(roundrect_rratio 0.25)
-			(net 70 "Net-(Q3-D)")
+			(net 70 "GNDD2")
 			(pintype "passive")
 		)
@@
 			(layers "F.Cu" "F.Mask" "F.Paste")
 			(roundrect_rratio 0.25)
-			(net 2 "GNDD")
+			(net 70 "GNDD2")
 			(pinfunction "S")
 			(pintype "passive")
@@
 			(layers "F.Cu" "F.Mask" "F.Paste")
 			(roundrect_rratio 0.25)
-			(net 70 "Net-(Q3-D)")
+			(net 70 "GNDD2")
 			(pintype "passive")
 		)
@@
 			(layers "F.Cu" "F.Mask" "F.Paste")
 			(roundrect_rratio 0.25)
-			(net 70 "Net-(Q3-D)")
+			(net 70 "GNDD2")
 			(pintype "passive")
 		)
@@
 	)
 	(segment
-		(start 104.4175 80.5)
-		(end 103.4175 80.5)
-		(width 0.25)
-		(layer "F.Cu")
-		(net 2)
-	)
-	(segment
 		(start 124.4175 54.5)
 		(end 124.4175 56.5)
@@
 		(net 2)
 	)
-	(segment
-		(start 103.4175 80.5)
-		(end 102.4175 79.5)
-		(width 0.25)
-		(layer "F.Cu")
-		(net 2)
-	)
 	(via
 		(at 87.4175 82.5)
@@
 	)
 	(via
-		(at 102.4175 79.5)
-		(size 0.6)
-		(drill 0.3)
-		(layers "F.Cu" "B.Cu")
-		(net 2)
-	)
-	(via
 		(at 108.28 64.5)
 		(size 0.6)
@@
 	)
 	(segment
-		(start 93.4175 62.5)
-		(end 93.7425 62.175)
+		(start 85.4175 63.101)
+		(end 72.0185 63.101)
 		(width 0.2)
 		(layer "F.Cu")
@@
 	)
 	(segment
-		(start 93.7425 62.175)
-		(end 96.0925 62.175)
+		(start 70.5925 61.675)
+		(end 66.4175 61.675)
 		(width 0.2)
 		(layer "F.Cu")
@@
 	)
 	(segment
-		(start 70.5925 61.675)
-		(end 72.0185 63.101)
+		(start 93.4175 62.5)
+		(end 93.7425 62.175)
 		(width 0.2)
 		(layer "F.Cu")
@@
 	)
 	(segment
-		(start 66.4175 61.675)
-		(end 70.5925 61.675)
+		(start 93.7425 62.175)
+		(end 96.0925 62.175)
 		(width 0.2)
 		(layer "F.Cu")
@@
 	(segment
 		(start 72.0185 63.101)
-		(end 84.4175 63.101)
+		(end 70.5925 61.675)
 		(width 0.2)
 		(layer "F.Cu")
@@
 	)
 	(via
-		(at 84.4175 63.101)
+		(at 85.4175 63.101)
 		(size 0.6)
 		(drill 0.3)
@@
 	)
 	(segment
-		(start 92.8165 63.101)
-		(end 93.4175 62.5)
+		(start 85.4175 63.101)
+		(end 92.8165 63.101)
 		(width 0.2)
 		(layer "B.Cu")
@@
 	)
 	(segment
-		(start 84.4175 63.101)
-		(end 92.8165 63.101)
+		(start 92.8165 63.101)
+		(end 93.4175 62.5)
 		(width 0.2)
 		(layer "B.Cu")
@@
 	)
 	(segment
+		(start 103.4175 80.5)
+		(end 102.4175 79.5)
+		(width 0.25)
+		(layer "F.Cu")
+		(net 70)
+	)
+	(segment
 		(start 72.4175 57.225)
 		(end 74.3175 57.225)
@@
 	)
 	(segment
+		(start 104.4175 80.5)
+		(end 103.4175 80.5)
+		(width 0.25)
+		(layer "F.Cu")
+		(net 70)
+	)
+	(segment
 		(start 74.3175 57.225)
 		(end 74.4175 57.325)
@@
 		(net 70)
 	)
+	(via
+		(at 102.4175 79.5)
+		(size 0.6)
+		(drill 0.3)
+		(layers "F.Cu" "B.Cu")
+		(net 70)
+	)
 	(segment
 		(start 78.4175 62.5)
@@
 	)
 	(segment
+		(start 102.4175 79.5)
+		(end 98.5175 79.5)
+		(width 0.25)
+		(layer "B.Cu")
+		(net 70)
+	)
+	(segment
 		(start 76.4175 60.5)
 		(end 78.4175 62.5)
 		(width 0.25)
 		(layer "B.Cu")
+		(net 70)
+	)
+	(segment
+		(start 98.5175 79.5)
+		(end 81.5175 62.5)
+		(width 0.25)
+		(layer "B.Cu")

Commit message: dev
Parts:
- removed the J3 at (68.4, 65.5)
- removed J7: USB_C_Receptacle_PowerOnly_6P, Connector_USB:USB_C_Receptacle_GCT_USB4135-GF-A_6P_TopMnt_Horizontal
- added D1: LED, LED_SMD:LED_1206_3216Metric_Pad1.42x1.75mm_HandSolder, B.Cu at (74.9, 64.5)
- added J5: Conn_01x06_Socket, Connector_JST:JST_PH_S6B-PH-K_1x06_P2.00mm_Horizontal, F.Cu at (62.4, 82.5)
- C13, R14, R15, R18, R19, R20: moved to B.Cu
- J3: renamed from J5; footprint Connector_JST:JST_PH_B2B-PH-K_1x02_P2.00mm_Vertical -> Connector_JST:JST_PH_S2B-PH-K_1x02_P2.00mm_Horizontal
- J4: renamed from J6; footprint Connector_JST:JST_PH_B6B-PH-K_1x06_P2.00mm_Vertical -> Connector_JST:JST_PH_S6B-PH-K_1x06_P2.00mm_Horizontal
- U2: value Ai-Thinker-Ra-02 -> Ra-01SCH-P
- moved R5 15.1 mm to (79.4, 64.5), turned to 180 degrees
- moved R1 10.5 mm to (68.4, 66.4), turned to -90 degrees
- moved SW1 9.83 mm to (70.4, 63.5)
- moved R8 8.25 mm to (66.4, 57.5), turned to 0 degrees
- moved C4 7.46 mm to (66.4, 66.4), turned to 90 degrees
- moved R14 5.34 mm to (66.4, 78.5), turned to 0 degrees
- moved J4 5.00 mm to (62.4, 58.5)
- moved C7 3.00 mm to (82.4, 48.5)
- moved J1 3.00 mm to (79.4, 50.0)
- moved C8 2.73 mm to (66.4, 59.5), turned to 0 degrees
- moved C5 2.00 mm to (107.4, 63.5)
- moved J3 1.45 mm to (93.4, 83.0), turned to 180 degrees
- moved R15 1.18 mm to (66.4, 76.5), turned to 0 degrees
Connections:
- J3 pad 1: VRAW -> +5V0
Routing:
- net +5V0: track 31.3 -> 71.3 mm, vias 2 -> 7
- net /INFO_LED: track 32.6 -> 16.7 mm, vias 3 -> 5
- net +3V3: track 155.8 -> 163.4 mm
- net VRAW: track 77.2 -> 70.1 mm
- net Net-(J4-Pin_5): track 35.8 -> 40.8 mm
- net /PB12: track 34.6 -> 39.6 mm
- net Net-(J3-Pin_2): track 5.38 -> 10.2 mm
- net Net-(J4-Pin_1): track 10.1 -> 5.52 mm, vias 2 -> 0
- net /SWDIO: track 41.2 -> 38.2 mm
- net /SWCLK: track 46.6 -> 43.6 mm
- net Net-(D1-A): track 4.83 -> 2.11 mm
- net GNDD: track 58.6 -> 56.0 mm, vias 37 -> 34
- net /RESET_PIN: track 61.3 -> 60.3 mm, vias 4 -> 5
- net Net-(J5-Pin_4): track 3.48 -> 3.09 mm, vias 1 -> 0
- net GNDD2: track 61.5 -> 61.9 mm, vias 3 -> 4
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Other:
- board size 80 x 42 mm -> 83 x 42 mm
- board text added: "BUZZER"
- board text added: "GND"
- board text added: "USB-C Power"
- board text removed: "G"

Commit message: lora setup done 70%
Routing:
- net GNDD2: track 61.9 -> 63.3 mm
Changed lines of the file:
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@@
 		(tags "resistor handsolder")
 		(property "Reference" "R9"
-			(at 3 0 180)
+			(at 2.662032 -0.055442 180)
 			(layer "F.SilkS")
 			(effects
@@
 		(tags "SOT TO_SOT_SMD")
 		(property "Reference" "Q2"
-			(at 3.0625 -0.05 180)
+			(at 2.703844 -0.008622 180)
 			(layer "F.SilkS")
 			(effects
@@
 	)
 	(segment
+		(start 76.505 83.5)
+		(end 77.505 82.5)
+		(width 0.25)
+		(layer "F.Cu")
+		(net 2)
+	)
+	(segment
 		(start 98.005 62.0875)
 		(end 98.4175 62.5)
@@
 	)
 	(segment
-		(start 77.505 82.5)
-		(end 77.505 83.5875)
-		(width 0.25)
-		(layer "F.Cu")
-		(net 2)
-	)
-	(segment
 		(start 93.634392 65.5)
 		(end 93.6925 65.558108)
@@
 	)
 	(segment
-		(start 77.505 83.5875)
-		(end 78.4175 84.5)
+		(start 75.4175 83.5)
+		(end 76.505 83.5)
 		(width 0.25)
 		(layer "F.Cu")
@@
 	)
 	(via
-		(at 78.4175 84.5)
+		(at 75.4175 83.5)
 		(size 0.6)
 		(drill 0.3)
@@
 	)
 	(segment
-		(start 78.4175 54.5)
-		(end 78.4175 55.5)
-		(width 0.25)
-		(layer "F.Cu")
-		(net 45)
-	)
-	(segment
-		(start 76.4175 54.5)
-		(end 76.4175 55.5)
-		(width 0.25)
-		(layer "F.Cu")
-		(net 45)
-	)
-	(segment
 		(start 72.4175 53.5)
 		(end 67.4175 48.5)
@@
 	)
 	(segment
-		(start 78.4175 54.5)
-		(end 77.4175 53.5)
-		(width 0.25)
-		(layer "F.Cu")
-		(net 45)
-	)
-	(segment
-		(start 72.4175 53.5)
-		(end 72.4175 55.5)
-		(width 0.25)
-		(layer "F.Cu")
-		(net 45)
-	)
-	(segment
 		(start 67.4175 48.5)
 		(end 62.4175 48.5)
@@
 	)
 	(segment
-		(start 76.4175 54.5)
-		(end 75.4175 53.5)
-		(width 0.25)
-		(layer "F.Cu")
-		(net 45)
-	)
-	(segment
 		(start 85.5785 55.339)
 		(end 86.4175 54.5)
@@
 	)
 	(via
-		(at 72.4175 55.5)
+		(at 90.4175 73.5)
 		(size 0.6)
 		(drill 0.3)
@@
 	)
 	(via
-		(at 76.4175 55.5)
+		(at 79.4175 53.5)
 		(size 0.6)
 		(drill 0.3)
@@
 	)
 	(via
-		(at 90.4175 73.5)
+		(at 72.4175 53.5)
 		(size 0.6)
 		(drill 0.3)
@@
 	)
 	(via
-		(at 78.4175 55.5)
+		(at 77.4175 53.5)
 		(size 0.6)
 		(drill 0.3)
@@
 	)
 	(via
-		(at 79.4175 53.5)
+		(at 92.4175 79.5)
 		(size 0.6)
 		(drill 0.3)
@@
 	)
 	(via
-		(at 92.4175 79.5)
+		(at 75.4175 53.5)
 		(size 0.6)
 		(drill 0.3)
@@
 	)
 	(segment
+		(start 78.4175 54.5)
+		(end 77.4175 53.5)
+		(width 0.25)
+		(layer "B.Cu")
+		(net 45)
+	)
+	(segment
 		(start 79.4175 53.5)
 		(end 83.4175 53.5)
@@
 	)
 	(segment
+		(start 76.4175 55.5)
+		(end 76.4175 54.5)
+		(width 0.25)
+		(layer "B.Cu")
+		(net 45)
+	)
+	(segment
 		(start 92.4175 76.5)
 		(end 90.4175 74.5)
@@
 	)
 	(segment
+		(start 72.4175 53.5)
+		(end 72.4175 55.5)
+		(width 0.25)
+		(layer "B.Cu")
+		(net 45)
+	)
+	(segment
 		(start 72.4175 55.5)
 		(end 71.33 55.5)
@@
 	)
 	(segment
+		(start 76.4175 54.5)
+		(end 75.4175 53.5)
+		(width 0.25)
+		(layer "B.Cu")
+		(net 45)
+	)
+	(segment
+		(start 78.4175 55.5)
+		(end 78.4175 54.5)
+		(width 0.25)
+		(layer "B.Cu")
+		(net 45)
+	)
+	(segment
 		(start 97.505 66.331739)
 		(end 97.505 67.5875)
@@
 	)
 	(segment
+		(start 110.4175 79.5875)
+		(end 109.37375 78.54375)
+		(width 0.2)
+		(layer "F.Cu")
+		(net 66)
+	)
+	(segment
 		(start 98.005 69.0875)
 		(end 98.005 67.5875)
@@
 	)
 	(via
-		(at 98.005 69.0875)
+		(at 109.37375 78.54375)
 		(size 0.6)
 		(drill 0.3)
@@
 	)
 	(via
-		(at 110.4175 79.5875)
+		(at 98.005 69.0875)
 		(size 0.6)
 		(drill 0.3)
@@
 	(segment
 		(start 103.532 72.702)
-		(end 110.4175 79.5875)
+		(end 109.37375 78.54375)
 		(width 0.2)
 		(layer "B.Cu")
@@
 	)
 	(segment
-		(start 87.4175 52.85)
-		(end 87.9175 52.85)
+		(start 75.4175 60.5)
+		(end 83.003286 60.5)
 		(width 0.25)
 		(layer "F.Cu")
@@
 	)
 	(segment
-		(start 104.4175 80.5)
-		(end 103.4175 80.5)
+		(start 87.4175 52.85)
+		(end 87.9175 52.85)
 		(width 0.25)
 		(layer "F.Cu")
@@
 	)
 	(segment
-		(start 87.3675 49.4875)
-		(end 87.3675 52.44187)
+		(start 104.4175 80.5)
+		(end 103.4175 80.5)
 		(width 0.25)
 		(layer "F.Cu")
@@
 	)
 	(segment
-		(start 83.003286 60.5)
-		(end 77.5925 60.5)
+		(start 74.4175 59.5)
+		(end 75.4175 60.5)
 		(width 0.25)
 		(layer "F.Cu")
@@
 	)
 	(segment
-		(start 77.5925 60.5)
-		(end 74.4175 57.325)
+		(start 87.3675 49.4875)
+		(end 87.3675 52.44187)
 		(width 0.25)
 		(layer "F.Cu")
@@
 	)
 	(segment
-		(start 83.010393 60.507107)
-		(end 83.003286 60.5)
+		(start 83.003286 60.5)
+		(end 83.010393 60.507107)
 		(width 0.25)
 		(layer "F.Cu")
@@
 	)
 	(via
-		(at 74.4175 57.325)
+		(at 74.4175 59.5)
 		(size 0.6)
 		(drill 0.3)
@@
 	)
 	(segment
-		(start 74.4175 57.325)
-		(end 72.5175 57.325)
+		(start 101.4175 76.5)
+		(end 101.4175 78.5)
 		(width 0.25)
 		(layer "B.Cu")
@@
 	)
 	(segment
-		(start 101.4175 76.5)
-		(end 101.4175 78.5)
+		(start 74.3175 57.225)
+		(end 74.4175 57.325)
+		(width 0.25)
+		(layer "B.Cu")
+		(net 68)
+	)
+	(segment
+		(start 72.4175 57.225)
+		(end 74.3175 57.225)
+		(width 0.25)
+		(layer "B.Cu")
+		(net 68)
+	)
+	(segment
+		(start 74.4175 59.5)
+		(end 74.4175 57.325)
 		(width 0.25)
 		(layer "B.Cu")
@@
 		(polygon
 			(pts
+				(xy 72.895634 52.966695) (xy 72.914024 54.226397) (xy 73.024363 54.741311) (xy 73.447328 55.201056)
+				(xy 74.100166 54.640167) (xy 74.826563 54.667752) (xy 75.387452 55.173471) (xy 75.966731 54.612582)
+				(xy 75.387452 54.005719) (xy 75.001266 53.656313) (xy 74.734614 52.828772) (xy 73.364574 52.828772)
+			)
+		)
+	)
+	(zone
+		(net 0)
+		(net_name "")
+		(layer "B.Cu")
+		(hatch edge 0.5)
+		(connect_pads
+			(clearance 0)
+		)
+		(min_thickness 0.25)
+		(filled_areas_thickness no)
+		(keepout
+			(tracks not_allowed)
+			(vias not_allowed)
+			(pads not_allowed)
+			(copperpour not_allowed)
+			(footprints allowed)
+		)
+		(placement
+			(enabled no)
+			(sheetname "/")
+		)
+		(fill
+			(thermal_gap 0.5)
+			(thermal_bridge_width 0.5)
+		)
+		(polygon
+			(pts
 				(xy 76.958099 56.380366) (xy 77.38942 55.830876) (xy 77.944819 56.457177) (xy 77.413054 57.024393)
 			)
@@
 			)
 		)
+	)
+	(zone
+		(net 0)
+		(net_name "")
+		(layer "B.Cu")
+		(hatch edge 0.5)
+		(connect_pads
+			(clearance 0)
+		)
+		(min_thickness 0.25)
+		(filled_areas_thickness no)
+		(keepout
+			(tracks not_allowed)
+			(vias not_allowed)
+			(pads not_allowed)
+			(copperpour not_allowed)
+			(footprints allowed)
+		)
+		(placement
+			(enabled no)
+			(sheetname "/")
+		)
+		(fill
+			(thermal_gap 0.5)
+			(thermal_bridge_width 0.5)
+		)
+		(polygon
+			(pts
+				(xy 77.421988 55.130562) (xy 77.881733 54.670817) (xy 77.060322 54.008784) (xy 76.821254 53.45709)
+				(xy 77.385737 52.990171) (xy 77.644232 53.192991) (xy 78.594447 54.159788) (xy 79.18292 54.941355)
+				(xy 79.256479 55.649362) (xy 79.100166 56.155081) (xy 78.989827 56.458513) (xy 79.256479 56.798724)
+				(xy 80.470206 56.026353) (xy 82.125288 54.049449) (xy 81.113849 53.9575) (xy 79.881733 53.985085)
+				(xy 79.146141 54.03106) (xy 78.907073 53.378222) (xy 78.640421 52.900087) (xy 75.780807 52.798943)
+				(xy 76.01068 53.516145) (xy 76.792246 54.545974) (xy 77.261186 55.106863)
+			)
+		)

Commit message: dev
Parts:
- removed D2, D3: SS34, Diode_SMD:D_SMA
- removed the R2 at (130.4, 73.9)
- added FB1: FerriteBead, Inductor_SMD:L_0603_1608Metric_Pad1.05x0.95mm_HandSolder, F.Cu at (128.4, 75.4)
- added R13: 10k, Resistor_SMD:R_0603_1608Metric_Pad0.98x0.95mm_HandSolder, B.Cu at (75.5, 68.5)
- added R14: 10k, Resistor_SMD:R_0603_1608Metric_Pad0.98x0.95mm_HandSolder, B.Cu at (68.4, 72.5)
- added SW2: SW_Push, Button_Switch_SMD:SW_Push_1TS009xxxx-xxxx-xxxx_6x6x5mm, B.Cu at (67.4, 49.5)
- added U3: TVS0500DRV, Package_SON:WSON-6-1EP_2x2mm_P0.65mm_EP1x1.6mm, B.Cu at (78.5, 75.8)
- added U5: TPS2116DRL, Package_TO_SOT_SMD:SOT-583-8, B.Cu at (75.7, 71.8)
- C10: value 470u -> C_Polarized 100uF electrolitic; footprint Capacitor_SMD:C_0805_2012Metric_Pad1.18x1.45mm_HandSolder -> Capacitor_SMD:CP_Elec_5x5.4
- moved C10 1.96 mm to (71.4, 80.5), turned to -90 degrees
- turned R19 to 90 degrees
- renumbered R11 to R10, R12 to R11, R13 to R12, R16 to R15, R17 to R16, R14 to R17, R15 to R18, R18 to R19, R3 to R2, R19 to R20, R20 to R21, R4 to R3, R5 to R4, R6 to R5, R7 to R6, R8 to R7, R9 to R8, R10 to R9, U3 to U4, U4 to U6
Connections:
- R10 pad 1: +3V3 -> VRAW
- R19 pad 1: +5V0 -> VRAW
- U1 pad 12: unconnected-(U1-PA2-Pad12) -> /LINK_BUTTON
- U1 pad 13: unconnected-(U1-PA3-Pad13) -> /LORA_BUSY
- U1 pad 18: /PB0 -> /LORA_DIO1
- U1 pad 19: unconnected-(U1-PB1-Pad19) -> /LORA_NRST
- U1 pad 42: unconnected-(U1-PB6-Pad42) -> INFO_SUPPLY
- U2 pad 1: GNDD -> unconnected-(U2-ANT-Pad1)
- U2 pad 10: unconnected-(U2-DIO4-Pad10) -> /LORA_BUSY
- U2 pad 3: Net-(Q1-D) -> Net-(U2-VDD)
- U2 pad 4: Net-(U2-~{RESET}) -> /LORA_NRST
- U2 pad 5: /PB0 -> unconnected-(U2-VCCPA-Pad5)
- U2 pad 6: unconnected-(U2-DIO1-Pad6) -> /LORA_DIO1
- U4 pad 2: GNDD -> VRAW
- U6 pad 2: GNDD2 -> VRAW
Routing:
- net /LINK_BUTTON: track 0.00 -> 53.3 mm, vias 0 -> 3
- net /LORA_BUSY: track 0.00 -> 44.0 mm, vias 0 -> 2
- net /LORA_DIO1: track 0.00 -> 43.0 mm, vias 0 -> 4
- net /PB0: track 41.0 -> 0.00 mm, vias 4 -> 0
- net /LORA_NRST: track 0.00 -> 39.4 mm, vias 0 -> 4
- net INFO_SUPPLY: track 0.00 -> 37.9 mm, vias 0 -> 4
- net +3V3: track 163.4 -> 143.1 mm
- net VRAW: track 70.1 -> 82.1 mm, vias 4 -> 6
- net Net-(J5-Pin_6): track 13.4 -> 22.7 mm
- net Net-(BT1-+): track 5.83 -> 14.0 mm
- net Net-(Q1-D): track 14.9 -> 9.07 mm
- net Net-(U2-VDD): track 0.00 -> 4.04 mm
- net Net-(U2-~{RESET}): track 3.03 -> 0.00 mm
- net Net-(U5-PR1): track 0.00 -> 2.52 mm
- net +5V0: track 71.3 -> 68.9 mm, vias 7 -> 6
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Other:
- board text added: "LINK"
