File: KiCAD/FlameSensorSender/FlameSensorSender.kicad_pcb (KiCad board)
At the start: 2 copper layers, 83 x 42 mm, 54 parts, among them J1 SWD, J3 JST-PH B2B-PH-K-S, J4 Sharp GP2Y1014AUOF, J5 Conn_01x06_Socket, Q1 AO3401A, Q2 AO3400A, Q3 AO3400A, SW1 SW_Push, SW2 SW_Push, U1 STM32F103C6Tx, U2 Ra-01SCH-P, U3 TVS0500DRV, U4 TPS63802DLAR, U5 TPS2116DRL, U6 TPS63802DLAR

Commit message: dev
Parts:
- removed the R15 at (93.4, 49.4)
- removed the R3 at (124.4, 75.4)
- added J2: SWD, Connector_PinHeader_2.54mm:PinHeader_2x02_P2.54mm_Vertical, B.Cu at (75.9, 65.5)
- added Q2: AO3400A, Package_TO_SOT_SMD:SOT-23-3, F.Cu at (122.4, 78.4)
- added Q5: AO3400A, Package_TO_SOT_SMD:SOT-23-3, F.Cu at (91.4, 49.6)
- added Q6: AO3401A, Package_TO_SOT_SMD:SOT-23-3, F.Cu at (87.4, 49.6)
- added R11: 10k,0603, Resistor_SMD:R_0603_1608Metric_Pad0.98x0.95mm_HandSolder, F.Cu at (82.4, 65.5)
- added R12: 10k,0603, Resistor_SMD:R_0603_1608Metric_Pad0.98x0.95mm_HandSolder, F.Cu at (82.5, 67.5)
- added R18: 10,0603, Resistor_SMD:R_0603_1608Metric_Pad0.98x0.95mm_HandSolder, F.Cu at (94.4, 49.6)
- added R2: 10k,0603, Resistor_SMD:R_0603_1608Metric_Pad0.98x0.95mm_HandSolder, F.Cu at (117.3, 75.5)
- added R7: 10k,0603, Resistor_SMD:R_0603_1608Metric_Pad0.98x0.95mm_HandSolder, F.Cu at (106.4, 80.5)
- C1, C2, C3, C5, C6: value 100n -> 100n,0603
- C10: renamed from C11; value 22u -> 22u,0603
- C13, C9: value 22u -> 22u,0603
- C4: value 105, 0603 -> 105,0603
- C8: value 220n -> 16V220u,alum 6.3x7.7; footprint Capacitor_SMD:C_0603_1608Metric_Pad1.08x0.95mm_HandSolder -> Capacitor_SMD:CP_Elec_6.3x7.7
- D1, R4: moved to F.Cu
- J7: renamed from J5; value Conn_01x06_Socket -> Conn_01x04_Socket; footprint Connector_JST:JST_PH_S6B-PH-K_1x06_P2.00mm_Horizontal -> Connector_JST:JST_PH_S4B-PH-K_1x04_P2.00mm_Horizontal
- L1, L2: value 470n -> 0.47u; footprint Inductor_SMD:L_Coilcraft_XxL4020 -> Footprints:INDC2016X120N
- Q3: value AO3400A -> AO3401A; footprint Package_TO_SOT_SMD:SOT-23 -> Package_TO_SOT_SMD:SOT-23-3
- Q4: renamed from Q2; footprint Package_TO_SOT_SMD:SOT-23 -> Package_TO_SOT_SMD:SOT-23-3
- R1: value 10k, 0603 -> 10k,0603
- R13: renamed from R10; value 100k Rpg -> 100k,0603
- R14: renamed from R11; value 511k Rfbt -> 511k,0603
- R15: renamed from R12; value 91k Rfbb -> 91k,0603
- R16: renamed from R13; value 10k -> 10k,0603
- R17: renamed from R14; value 10k -> 10k,0603
- R19: renamed from R16; value 470k,0603 -> 10k,0603
- R20: renamed from R17; value 5.1k -> 5.1k,0603
- R21: renamed from R18; value 5.1k -> 5.1k,0603
- R22: renamed from R19; value 100k Rpg -> 100k,0603; moved to F.Cu
- R23: renamed from R20; value 806k Rfbt -> 806k,0603
- R24: renamed from R21; value 91k Rfbb -> 91k,0603
- R3: renamed from R2; value 1k,0603 -> 10,0603
- R5: value 220 -> 220,0603
- R6: value 330 -> 330,0603
- R8: renamed from R9; value 1k,0603 -> 10,0603
- R9: renamed from R7; value 150 -> 150,0603
- moved D1 43.6 mm to (118.4, 62.5)
- moved R4 41.0 mm to (120.4, 66.5), turned to 0 degrees
- moved Q3 35.5 mm to (102.5, 80.6)
- moved C8 20.3 mm to (66.4, 79.8), turned to -90 degrees
- moved R20 6.00 mm to (66.4, 72.5), turned to 90 degrees
- moved R22 5.53 mm to (82.4, 52.6), turned to -90 degrees
- moved Q4 5.06 mm to (110.4, 80.6)
- moved R21 4.47 mm to (64.4, 72.5), turned to 90 degrees
- moved R19 4.18 mm to (88.4, 46.5), turned to 180 degrees
- moved Q1 4.00 mm to (117.4, 78.4)
- moved R8 4.00 mm to (114.4, 80.5)
- moved R23 3.00 mm to (79.4, 56.4)
- moved J7 2.24 mm to (61.4, 80.5)
- moved R10 2.24 mm to (98.4, 80.5)
- moved R6 2.00 mm to (103.4, 49.5)
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- renumbered C10 to C11, J3 to J6, R8 to R10
Connections:
- net /INFO_BUZZER renamed /BUZZER
- net /LORA EN renamed /MOSFET_GATE_LORA
- net /PB12 renamed /SENSOR_LED
- net /SENSOR DATA renamed /SENSOR DATA Vo
- net Net-(J4-Pin_5) renamed /Vo
- C12 pad 1: VRAW -> Net-(Q6-D)
- C12 pad 2: GNDD2 -> GNDD
- C13 pad 2: GNDD2 -> GNDD
- C8 pad 1: Net-(J4-Pin_1) -> /V-LED
- J4 pad 1: Net-(J4-Pin_1) -> /V-LED
- J6 pad 1: +5V0 -> Net-(J6-Pin_1)
- J6 pad 2: Net-(J3-Pin_2) -> GNDD
- J7 pad 2: unconnected-(J5-Pin_2-Pad2) -> Net-(J7-Pin_2)
- J7 pad 3: Net-(J5-Pin_3) -> Net-(J7-Pin_3)
- J7 pad 4: Net-(J5-Pin_4) -> Net-(J7-Pin_4)
- Q3 pad 2: GNDD -> +5V0
- Q3 pad 3: GNDD2 -> Net-(Q3-D)
- Q4 pad 2: GNDD2 -> GNDD
- Q4 pad 3: Net-(Q2-D) -> Net-(Q3-G)
- R10 pad 1: Net-(Q2-D) -> Net-(Q3-D)
- R10 pad 2: Net-(J3-Pin_2) -> Net-(J6-Pin_1)
- R16 pad 1: Net-(J5-Pin_6) -> Net-(J7-Pin_4)
- R17 pad 2: Net-(J5-Pin_6) -> Net-(J7-Pin_4)
- R19 pad 1: Net-(Q3-G) -> Net-(Q5-D)
- R19 pad 2: GNDD -> VRAW
- R20 pad 1: Net-(J5-Pin_3) -> Net-(J7-Pin_2)
- R21 pad 1: Net-(J5-Pin_4) -> Net-(J7-Pin_3)
- R22 pad 1: VRAW -> Net-(Q6-D)
- R24 pad 2: GNDD2 -> GNDD
- R3 pad 2: Net-(Q1-G) -> Net-(Q2-G)
- R9 pad 1: Net-(J4-Pin_1) -> +5V0
- R9 pad 2: +5V0 -> /V-LED
- U1 pad 11: unconnected-(U1-PA1-Pad11) -> VCC_BAT
- U1 pad 21: SENSOR EN -> MOSFET_GATE_SENSOR
- U1 pad 28: /INFO_LED -> unconnected-(U1-PB15-Pad28)
- U1 pad 3: unconnected-(U1-PC14-Pad3) -> /INFO_LED
- U1 pad 30: unconnected-(U1-PA9-Pad30) -> /USART1_TX
- U1 pad 31: unconnected-(U1-PA10-Pad31) -> /USART1_RX
- U5 pad 3: Net-(J5-Pin_6) -> Net-(J7-Pin_4)
- U5 pad 5: Net-(J5-Pin_6) -> Net-(J7-Pin_4)
- U6 pad 1: VRAW -> Net-(Q6-D)
- U6 pad 10: VRAW -> Net-(Q6-D)
- U6 pad 2: VRAW -> Net-(Q6-D)
- U6 pad 3: GNDD2 -> GNDD
- U6 pad 8: GNDD2 -> GNDD
Routing:
- net GNDD2: track 62.8 -> 0.00 mm, vias 4 -> 0
- net VCC_BAT: track 0.00 -> 53.0 mm, vias 0 -> 4
- net Net-(J7-Pin_4): track 0.00 -> 26.9 mm
- net /V-LED: track 0.00 -> 25.4 mm, vias 0 -> 2
- net Net-(J5-Pin_6): track 22.7 -> 0.00 mm
- net /USART1_TX: track 0.00 -> 19.2 mm, vias 0 -> 2
- net /USART1_RX: track 0.00 -> 18.3 mm, vias 0 -> 2
- net GNDD: track 58.3 -> 75.5 mm, vias 40 -> 45
- net SENSOR EN: track 11.3 -> 0.00 mm
- net MOSFET_GATE_SENSOR: track 0.00 -> 10.7 mm
- net Net-(J3-Pin_2): track 10.2 -> 0.00 mm
- net +5V0: track 68.9 -> 78.8 mm, vias 6 -> 4
- net Net-(Q6-D): track 0.00 -> 9.89 mm
- net +3V3: track 143.1 -> 135.3 mm, vias 2 -> 4
- net Net-(J7-Pin_2): track 0.00 -> 7.16 mm
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- added copper zone on B.Cu, net Net-(BT1-+)
- added copper zone on B.Cu, net Net-(J7-Pin_4)
Other:
- board text added: "+5V0"
- board text added: "ANT"
- board text added: "BUSY"
- board text added: "DIO1"
- board text added: "DIO2"
- board text added: "DIO3"
- board text added: "G"
- board text added: "INFO LED"
- board text added: "L1"
- board text added: "MISO"
- board text added: "MOSI"
- board text added: "NSS"
- board text added: "RESET"
- board text added: "RF_EN"
- board text added: "RX"
- board text added: "SCK"
- board text added: "TX"
- board text added: "V-LED"
- board text added: "VCCPA"
- board text removed: "LED"
