File: KiCAD/FlameSensorSender/FlameSensorSender.kicad_sch (KiCad schematic)
At the start: 39 parts, among them J1 Sharp GP2Y1014AUOF, J2 SWD, Q1 AO3400A, Q2 AO3400A, SW1 SW_Push, U1 STM32F103C6Tx, U2 Ai-Thinker-Ra-02, U3 TPS63802DLAR, U4 TPS63802DLAR

Commit message: dev
Parts:
- added J3: USB_C_Receptacle_PowerOnly_6P, symbol Connector:USB_C_Receptacle_PowerOnly_6P
- Q1, Q2: value AO3400A -> AO3401A; footprint Package_TO_SOT_SMD:SOT-23 -> Package_TO_SOT_SMD:SOT-23_Handsoldering; symbol Transistor_FET:AO3400A -> Transistor_FET:AO3401A
Connections:
- new net: J3.A12 (GND), J3.B12 (GND)
- new net: J3.A9 (VBUS), J3.B9 (VBUS)
Changed lines of the file:
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@@
 	)
 	(symbol
-		(lib_id "Transistor_FET:AO3400A")
+		(lib_id "Transistor_FET:AO3401A")
 		(at 144.78 57.15 90)
 		(unit 1)
@@
 			)
 		)
-		(property "Value" "AO3400A"
+		(property "Value" "AO3401A"
 			(at 144.78 50.8 90)
 			(effects
@@
 			)
 		)
-		(property "Footprint" "Package_TO_SOT_SMD:SOT-23"
+		(property "Footprint" "Package_TO_SOT_SMD:SOT-23_Handsoldering"
 			(at 146.685 52.07 0)
 			(effects
@@
 			)
 		)
-		(property "Datasheet" "http://www.aosmd.com/pdfs/datasheet/AO3400A.pdf"
+		(property "Datasheet" "http://www.aosmd.com/pdfs/datasheet/AO3401A.pdf"
 			(at 148.59 52.07 0)
 			(effects
@@
 			)
 		)
-		(property "Description" "30V Vds, 5.7A Id, N-Channel MOSFET, SOT-23"
+		(property "Description" "-4.0A Id, -30V Vds, P-Channel MOSFET, SOT-23"
 			(at 144.78 57.15 0)
 			(effects
@@
 	)
 	(symbol
+		(lib_id "Connector:USB_C_Receptacle_PowerOnly_6P")
+		(at 311.15 77.47 0)
+		(unit 1)
+		(exclude_from_sim no)
+		(in_bom yes)
+		(on_board yes)
+		(dnp no)
+		(fields_autoplaced yes)
+		(property "Reference" "J3"
+			(at 311.15 59.69 0)
+			(effects
+				(font
+					(size 1.27 1.27)
+				)
+			)
+		)
+		(property "Value" "USB_C_Receptacle_PowerOnly_6P"
+			(at 311.15 62.23 0)
+			(effects
+				(font
+					(size 1.27 1.27)
+				)
+			)
+		)
+		(property "Footprint" ""
+			(at 314.96 74.93 0)
+			(effects
+				(font
+					(size 1.27 1.27)
+				)
+				(hide yes)
+			)
+		)
+		(property "Datasheet" "https://www.usb.org/sites/default/files/documents/usb_type-c.zip"
+			(at 311.15 77.47 0)
+			(effects
+				(font
+					(size 1.27 1.27)
+				)
+				(hide yes)
+			)
+		)
+		(property "Description" "USB Power-Only 6P Type-C Receptacle connector"
+			(at 311.15 77.47 0)
+			(effects
+				(font
+					(size 1.27 1.27)
+				)
+				(hide yes)
+			)
+		)
+		(pin "B9"
+		)
+		(pin "S1"
+		)
+		(pin "B12"
+		)
+		(pin "A12"
+		)
+		(pin "A9"
+		)
+		(pin "A5"
+		)
+		(pin "B5"
+		)
+		(instances
+			(project ""
+				(path "/a1d9ab92-440a-49d1-ae86-3051bc03dcb3"
+					(reference "J3")
+					(unit 1)
+				)
+			)
+		)
+	)
+	(symbol
 		(lib_id "Device:C")
 		(at 52.07 36.83 180)
@@
 	)
 	(symbol
-		(lib_id "Transistor_FET:AO3400A")
+		(lib_id "Transistor_FET:AO3401A")
 		(at 177.8 57.15 90)
 		(unit 1)
@@
 			)
 		)
-		(property "Value" "AO3400A"
+		(property "Value" "AO3401A"
 			(at 177.8 50.8 90)
 			(effects
@@
 			)
 		)
-		(property "Footprint" "Package_TO_SOT_SMD:SOT-23"
+		(property "Footprint" "Package_TO_SOT_SMD:SOT-23_Handsoldering"
 			(at 179.705 52.07 0)
 			(effects
@@
 			)
 		)
-		(property "Datasheet" "http://www.aosmd.com/pdfs/datasheet/AO3400A.pdf"
+		(property "Datasheet" "http://www.aosmd.com/pdfs/datasheet/AO3401A.pdf"
 			(at 181.61 52.07 0)
 			(effects
@@
 			)
 		)
-		(property "Description" "30V Vds, 5.7A Id, N-Channel MOSFET, SOT-23"
+		(property "Description" "-4.0A Id, -30V Vds, P-Channel MOSFET, SOT-23"
 			(at 177.8 57.15 0)
 			(effects

Commit message: dev
Parts:
- removed BT1: CR123A 3V, Battery:BatteryHolder_Keystone_2462_2xAA, symbol Device:Battery_Cell
- removed C12, C7, C8, C9: 22u, Capacitor_SMD:C_0603_1608Metric_Pad1.08x0.95mm_HandSolder, symbol Device:C
- removed D1, D2: 1N5819, Diode_SMD:D_0805_2012Metric_Pad1.15x1.40mm_HandSolder, symbol Diode:1N5819
- removed J3: USB_C_Receptacle_PowerOnly_6P, symbol Connector:USB_C_Receptacle_PowerOnly_6P
- removed L1, L2: 470n, Inductor_SMD:L_Coilcraft_XxL4020, symbol Device:L
- removed Q2: AO3401A, Package_TO_SOT_SMD:SOT-23_Handsoldering, symbol Transistor_FET:AO3401A
- removed R11: 100k Rpg, Resistor_SMD:R_0603_1608Metric_Pad0.98x0.95mm_HandSolder, symbol Device:R
- removed R12: 806k Rfbt, Resistor_SMD:R_0603_1608Metric_Pad0.98x0.95mm_HandSolder, symbol Device:R
- removed R13, R6: 91k Rfbb, Resistor_SMD:R_0603_1608Metric_Pad0.98x0.95mm_HandSolder, symbol Device:R
- removed R5: 511k Rfbt, Resistor_SMD:R_0603_1608Metric_Pad0.98x0.95mm_HandSolder, symbol Device:R
- removed R7: 10k, Resistor_SMD:R_0805_2012Metric_Pad1.20x1.40mm_HandSolder, symbol Device:R
- removed U3, U4: TPS63802DLAR, Footprints:VREG_TPS63802DLAR, symbol Custom_library:TPS63802DLAR
- C1, C2, C3, C6: footprint Capacitor_SMD:C_0805_2012Metric_Pad1.18x1.45mm_HandSolder -> Capacitor_SMD:C_0603_1608Metric_Pad1.08x0.95mm_HandSolder
- C5: renamed from C4; footprint Capacitor_SMD:C_0805_2012Metric_Pad1.18x1.45mm_HandSolder -> Capacitor_SMD:C_0603_1608Metric_Pad1.08x0.95mm_HandSolder
- C7: renamed from C11; footprint Capacitor_SMD:C_0805_2012Metric_Pad1.18x1.45mm_HandSolder -> Capacitor_SMD:C_0603_1608Metric_Pad1.08x0.95mm_HandSolder
- C8: renamed from C10; footprint Capacitor_SMD:C_0805_2012Metric_Pad1.18x1.45mm_HandSolder -> Capacitor_SMD:C_0603_1608Metric_Pad1.08x0.95mm_HandSolder
- R2: footprint Resistor_SMD:R_0805_2012Metric_Pad1.20x1.40mm_HandSolder -> Resistor_SMD:R_0201_0603Metric_Pad0.64x0.40mm_HandSolder
- R3: value 10k -> 1k,0603; footprint Resistor_SMD:R_0805_2012Metric_Pad1.20x1.40mm_HandSolder -> Resistor_SMD:R_0201_0603Metric_Pad0.64x0.40mm_HandSolder
- R4: value 100k Rpg -> 470k,0603; footprint Resistor_SMD:R_0603_1608Metric_Pad0.98x0.95mm_HandSolder -> Resistor_SMD:R_0201_0603Metric_Pad0.64x0.40mm_HandSolder
- R5: renamed from R8; footprint Resistor_SMD:R_0805_2012Metric_Pad1.20x1.40mm_HandSolder -> Resistor_SMD:R_0603_1608Metric_Pad0.98x0.95mm_HandSolder
- R6: renamed from R9; footprint Resistor_SMD:R_0805_2012Metric_Pad1.20x1.40mm_HandSolder -> Resistor_SMD:R_0603_1608Metric_Pad0.98x0.95mm_HandSolder
- R7: renamed from R10; footprint Resistor_SMD:R_0805_2012Metric_Pad1.20x1.40mm_HandSolder -> Resistor_SMD:R_0603_1608Metric_Pad0.98x0.95mm_HandSolder
- renumbered C5 to C4, J2 to J1, J1 to J2
Connections:
- net LORA EN: now also R3.1; no longer R3.2
- net at Q1.1 (G): now also R3.2, R4.1; no longer R3.1
- net +3V3: now reaches R4.2
- net +3V3: now also C1.1, C2.1, C3.1, C5.1, C6.1, C7.2, J1.1 (Pin_1), Q1.2 (S), R1.1, R2.2, U1.1 (VBAT), U1.24 (VDD), U1.36 (VDD), U1.48 (VDD), U1.9 (VDDA)
- net at U2.3 (VDD): now also Q1.3 (D)
- net +5V0: now reaches J2.6 (Pin_6), R7.2
- removed net +3V3 regulated: C1.1, C2.1, C3.1, C5.1, C6.1, C7.2, J1.1 (Pin_1), Q1.2 (S), R1.1, R2.2, R4.1, U1.1 (VBAT), U1.24 (VDD), U1.36 (VDD), U1.48 (VDD), U1.9 (VDDA)
Other:
- added sheet Power (power.kicad_sch)
- note removed: "AA Battery Li 2pcs."
- note removed: "DC-DC BUCK-BOOST converter, Vin 1V3 - 5V5, Vout 3V3"
- note removed: "DC-DC BUCK-BOOST converter, Vin 1V3 - 5V5, Vout 5V0"
- moved on the sheet: C4, C7, C8, J1, J2, R1, R2, R3, R5, R6, R7, SW1

Commit message: dev
Parts:
- added BZ1: Buzzer, symbol Device:Buzzer
- added D1: LED, LED_THT:LED_D5.0mm, symbol Device:LED
- added J2, J4: JST-PH PHR-2, symbol Connector:Conn_01x02_Pin
- added J3, J5: JST-PH B2B-PH-K-S, Connector_JST:JST_PH_B2B-PH-K_1x02_P2.00mm_Vertical, symbol Connector:Conn_01x02_Socket
- added R3: 220,0603, Resistor_SMD:R_0603_1608Metric_Pad0.98x0.95mm_HandSolder, symbol Device:R
- added R6: 110,0603, Resistor_SMD:R_0603_1608Metric_Pad0.98x0.95mm_HandSolder, symbol Device:R
- C7: value 104, 0805 -> 104,0603
- J6: renamed from J2; footprint Connector_JST:JST_PH_S6B-PH-K_1x06_P2.00mm_Horizontal -> Connector_JST:JST_PH_B6B-PH-K_1x06_P2.00mm_Vertical
- Q1: footprint Package_TO_SOT_SMD:SOT-23_Handsoldering -> Package_TO_SOT_SMD:SOT-23-3
- R2: footprint Resistor_SMD:R_0201_0603Metric_Pad0.64x0.40mm_HandSolder -> Resistor_SMD:R_0603_1608Metric_Pad0.98x0.95mm_HandSolder
- R4: renamed from R3; footprint Resistor_SMD:R_0201_0603Metric_Pad0.64x0.40mm_HandSolder -> Resistor_SMD:R_0603_1608Metric_Pad0.98x0.95mm_HandSolder
- R5: renamed from R4; footprint Resistor_SMD:R_0201_0603Metric_Pad0.64x0.40mm_HandSolder -> Resistor_SMD:R_0603_1608Metric_Pad0.98x0.95mm_HandSolder
- renumbered R5 to R7, R6 to R8, R7 to R9
Connections:
- net GNDD: now also J3.2 (Pin_2), J5.2 (Pin_2)
- net LORA_SCK: now reaches U1.15 (PA5), U2.12 (SCK)
- net LORA_MISO: now reaches U1.16 (PA6), U2.13 (MISO)
- net LORA_MOSI: now reaches U1.17 (PA7), U2.14 (MOSI)
- net LORA_NSS: now reaches U1.14 (PA4), U2.15 (~{NSS})
- net INFO_LED: now reaches U1.28 (PB15)
- net INFO_LED: now also R3.1
- net INFO_BUZZER: now reaches U1.38 (PA15)
- net INFO_BUZZER: now also R6.1
- new net: D1.1 (K), J2.2 (Pin_2)
- new net: D1.2 (A), J2.1 (Pin_1)
- new net: BZ1.1 (+), J4.1 (Pin_1)
- new net: BZ1.2 (-), J4.2 (Pin_2)
- new net: J5.1 (Pin_1), R6.2
- new net: J3.1 (Pin_1), R3.2
- no-connect marks 32 -> 30
Other:
- note added: "EXTERNAL"
- note added: "External BUZZER"
- note added: "External LED Indicator"
- moved on the sheet: C8, J6, R5, R7, R8, R9

Commit message: dev
Parts:
- added BZ1: Buzzer, Buzzer_Beeper:Buzzer_12x9.5RM7.6, symbol Device:Buzzer
- added Q1: AO3400A, Package_TO_SOT_SMD:SOT-23, symbol Transistor_FET:AO3400A
- added R3: 1k,0603, Resistor_SMD:R_0603_1608Metric_Pad0.98x0.95mm_HandSolder, symbol Device:R
- renumbered BZ1 to BZ2, Q1 to Q2, R9 to R10, R3 to R6, R6 to R9
Connections:
- net +5V0: now also BZ1.1 (+)
- net GNDD: now also Q1.2 (S)
- new net: Q1.1 (G), R3.2
- new net: BZ1.2 (-), Q1.3 (D)

Commit message: dev
Parts:
- removed BZ2: Buzzer, symbol Device:Buzzer
- R9: value 110,0603 -> 330,0603
- renumbered Q2 to Q1, Q1 to Q2, R3 to R10, R4 to R3, R5 to R4, R6 to R5, R7 to R6, R8 to R7, R10 to R8
Connections:
- net +5V0: no longer BZ1.1 (+)
- net GNDD: no longer J5.2 (Pin_2)
- net INFO_BUZZER: now also R10.2; no longer R9.1
- net at R10.1: now also Q2.1 (G)
- net at J4.1 (Pin_1): now also BZ1.1 (+)
- net at J4.2 (Pin_2): now also BZ1.2 (-)
- net at Q2.3 (D): now also R9.1; no longer BZ1.2 (-)
- net at R9.2: now also J5.2 (Pin_2); no longer J5.1 (Pin_1)
- new net VRAW: J5.1 (Pin_1)
Other:
- moved on the sheet: BZ1, J4, J5, Q2, R10, R9

Commit message: dev
Parts:
- U2: value Ai-Thinker-Ra-02 -> Ra-01SCH-P
Connections:
- net GNDD: no longer Q2.2 (S)
- new net GNDD2: Q2.2 (S)
Changed lines of the file:
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@@
+		)
+	)
+	(global_label "GNDD2"
+		(shape input)
+		(at 274.32 119.38 0)
+		(fields_autoplaced yes)
+		(effects
+			(font
+				(size 1.27 1.27)
+			)
+			(justify left)
+		)
+		(property "Intersheetrefs" "${INTERSHEET_REFS}"
+			(at 280.9849 119.38 0)
+			(effects
+				(font
+					(size 1.27 1.27)
+				)
+				(justify left)
+				(hide yes)
+			)
 		)
 	)
@@
 			)
 		)
-		(property "Value" "Ai-Thinker-Ra-02"
+		(property "Value" "Ra-01SCH-P"
 			(at 108.966 56.896 0)
 			(effects
@@
 					(unit 1)
 				)
-			)
-		)
-	)
-	(symbol
-		(lib_id "power:GNDD")
-		(at 274.32 119.38 90)
-		(unit 1)
-		(exclude_from_sim no)
-		(in_bom yes)
-		(on_board yes)
-		(dnp no)
-		(fields_autoplaced yes)
-		(property "Reference" "#PWR014"
-			(at 280.67 119.38 0)
-			(effects
-				(font
-					(size 1.27 1.27)
-				)
-				(hide yes)
-			)
-		)
-		(property "Value" "GNDD"
-			(at 278.13 119.38 90)
-			(effects
-				(font
-					(size 1.27 1.27)
-				)
-				(justify right)
-			)
-		)
-		(property "Footprint" ""
-			(at 274.32 119.38 0)
-			(effects
-				(font
-					(size 1.27 1.27)
-				)
-				(hide yes)
-			)
-		)
-		(property "Datasheet" ""
-			(at 274.32 119.38 0)
-			(effects
-				(font
-					(size 1.27 1.27)
-				)
-				(hide yes)
-			)
-		)
-		(property "Description" "Power symbol creates a global label with name \"GNDD\" , digital ground"
-			(at 274.32 119.38 0)
-			(effects
-				(font
-					(size 1.27 1.27)
-				)
-				(hide yes)
-			)
-		)
-		(pin "1"
-		)
-		(instances
-			(project "FlameSensorSender"
-				(path "/a1d9ab92-440a-49d1-ae86-3051bc03dcb3"
-					(reference "#PWR014")
-					(unit 1)
-				)
