File: KiCAD/FlameSensorSender/FlameSensorSender.kicad_sch (KiCad schematic)
At the start: 29 parts, among them J1 SWD, J2 JST-PH PHR-2, J3 JST-PH B2B-PH-K-S, J4 Sharp GP2Y1014AUOF, Q1 AO3401A, Q2 AO3400A, SW1 SW_Push, U1 STM32F103C6Tx, U2 Ra-01SCH-P

Commit message: lora setup done 70%
Other:
- note added: "Optical dust/smoke sensor Sharp"
- note removed: "Optical smole dust/smoke sensor Sharp"
Changed lines of the file:
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@@
 		)
 	)
-	(text "Optical smole dust/smoke sensor Sharp"
+	(text "Optical dust/smoke sensor Sharp"
 		(exclude_from_sim no)
 		(at 246.126 27.432 0)
