File: KiCAD/FlameSensorSender/FlameSensorSender.kicad_sch (KiCad schematic)
At the start: 30 parts, among them J1 SWD, J2 JST-PH PHR-2, J3 JST-PH B2B-PH-K-S, J4 Sharp GP2Y1014AUOF, Q1 AO3401A, Q2 AO3400A, SW1 SW_Push, SW2 SW_Push, U1 STM32F103C6Tx, U2 Ra-01SCH-P

Commit message: dev
Parts:
- removed R3: 470k,0603, Resistor_SMD:R_0603_1608Metric_Pad0.98x0.95mm_HandSolder, symbol Device:R
- added J2: SWD, Connector_PinHeader_2.54mm:PinHeader_2x02_P2.54mm_Vertical, symbol Connector_Generic:Conn_02x02_Counter_Clockwise
- added J3: Conn_01x06_Pin, Connector_JST:JST_PH_S6B-PH-K_1x06_P2.00mm_Horizontal, symbol Connector:Conn_01x06_Pin
- added Q2: AO3400A, Package_TO_SOT_SMD:SOT-23-3, symbol Transistor_FET:AO3400A
- added Q3: AO3401A, Package_TO_SOT_SMD:SOT-23-3, symbol Transistor_FET:AO3401A
- added R2, R7: 10k,0603, Resistor_SMD:R_0603_1608Metric_Pad0.98x0.95mm_HandSolder, symbol Device:R
- BZ1: value Buzzer -> SFM-20B
- C1, C2, C3, C5, C6: value 100n -> 100n,0603
- C4: value 105, 0603 -> 105,0603
- C8: value 220n -> 16V220u,alum 6.3x7.7; footprint Capacitor_SMD:C_0603_1608Metric_Pad1.08x0.95mm_HandSolder -> Capacitor_SMD:CP_Elec_6.3x7.7
- Q4: renamed from Q2; footprint Package_TO_SOT_SMD:SOT-23 -> Package_TO_SOT_SMD:SOT-23-3
- R1: value 10k, 0603 -> 10k,0603
- R3: renamed from R2; value 1k,0603 -> 10,0603
- R5: value 220 -> 220,0603
- R6: value 330 -> 330,0603
- R8: renamed from R9; value 1k,0603 -> 10,0603
- R9: renamed from R7; value 150 -> 150,0603
- renumbered J2 to J5, J3 to J6, R8 to R10
Connections:
- net GNDD2 is gone; now on net GNDD: Q4.2 (S)
- net +3V3: now also R2.2
- net +5V0: now also R9.1, Q3.2 (S), R7.1; no longer J6.1 (Pin_1), R9.2
- net GNDD: now also J6.2 (Pin_2), J2.1 (Pin_1), Q2.2 (S)
- net INFO_LED: now also U1.3 (PC14); no longer U1.28 (PB15)
- net at R3.2: now also Q2.1 (G); no longer Q1.1 (G)
- net Vo: now reaches J4.5 (Pin_5), R5.2
- net V-LED: now reaches C8.1, J4.1 (Pin_1)
- net V-LED: now also R9.2; no longer R9.1
- net at R10.2: now also J6.1 (Pin_1); no longer J6.2 (Pin_2)
- net at Q4.3 (D): now also Q3.1 (G), R7.2; no longer R10.1
- net VCC_BAT: now reaches U1.11 (PA1)
- net USART1_TX: now reaches U1.30 (PA9)
- net USART1_TX: now also J2.2 (Pin_2)
- net USART1_RX: now reaches U1.31 (PA10)
- net USART1_RX: now also J2.4 (Pin_4)
- net INFO_BUZZER renamed BUZZER
- net LORA EN renamed MOSFET_GATE_LORA
- net PB12 renamed SENSOR_LED
- net SENSOR DATA renamed SENSOR DATA Vo
- net SENSOR EN renamed MOSFET_GATE_SENSOR
- new net: Q1.1 (G), Q2.3 (D), R2.1
- new net: Q3.3 (D), R10.1
- no-connect marks 26 -> 30
Other:
- note added: "USART Interface"
- moved on the sheet: BZ1, C8, D1, J4, J5, J6, Q4, R10, R3, R4, R5, R6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

Commit message: dev
Parts:
- U1: value STM32F103C6Tx -> STM32F103C8Tx
Changed lines of the file:
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@@
 			)
 		)
-		(property "Value" "STM32F103C6Tx"
+		(property "Value" "STM32F103C8Tx"
 			(at 55.88 89.662 0)
 			(effects
