File: KiCAD/FlameSensorSender/power.kicad_sch (KiCad schematic)
At the start: 27 parts, among them J5 Conn_01x06_Socket, J6 Conn_01x06_Pin, J7 6 Pin USB-C Type USB Connecto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, Q3 AO3400A, U3 TPS63802DLAR, U4 TPS2116DRL, U5 TPS63802DLAR

Commit message: dev
Parts:
- removed Q3: AO3400A, Package_TO_SOT_SMD:SOT-23, symbol Transistor_FET:AO3400A
- removed R17: 1k,0603, Resistor_SMD:R_0603_1608Metric_Pad0.98x0.95mm_HandSolder, symbol Device:R
- added Q5: AO3400A, Package_TO_SOT_SMD:SOT-23-3, symbol Transistor_FET:AO3400A
- added Q6: AO3401A, Package_TO_SOT_SMD:SOT-23-3, symbol Transistor_FET:AO3401A
- added R11, R12: 10k,0603, Resistor_SMD:R_0603_1608Metric_Pad0.98x0.95mm_HandSolder, symbol Device:R
- added R18: 10,0603, Resistor_SMD:R_0603_1608Metric_Pad0.98x0.95mm_HandSolder, symbol Device:R
- added U3: TVS0500DRV, Package_SON:WSON-6-1EP_2x2mm_P0.65mm_EP1x1.6mm, symbol Power_Protection:TVS0500DRV
- C10: renamed from C11; value 22u -> 22u,0603
- C12, C13, C9: value 22u -> 22u,0603
- J7: renamed from J5; value Conn_01x06_Socket -> Conn_01x04_Socket; footprint Connector_JST:JST_PH_S6B-PH-K_1x06_P2.00mm_Horizontal -> Connector_JST:JST_PH_S4B-PH-K_1x04_P2.00mm_Horizontal; symbol Connector:Conn_01x06_Socket -> Connector:Conn_01x04_Socket
- J8: renamed from J6; value Conn_01x06_Pin -> Conn_01x04_Pin; symbol Connector:Conn_01x06_Pin -> Connector:Conn_01x04_Pin
- L1, L2: value 470n -> 0.47u; footprint Inductor_SMD:L_Coilcraft_XxL4020 -> Footprints:INDC2016X120N
- R13: renamed from R11; value 100k Rpg -> 100k,0603
- R14: renamed from R12; value 511k Rfbt -> 511k ~ 510k,0603
- R15: renamed from R13; value 91k Rfbb -> 91k,0603
- R16: renamed from R10; value 10k -> 10k,0603
- R17: renamed from R14; value 10k -> 10k,0603
- R19: renamed from R18; value 470k,0603 -> 10k,0603
- R20: renamed from R15; value 5.1k -> 5.1k,0603
- R21: renamed from R16; value 5.1k -> 5.1k,0603
- R22: renamed from R19; value 100k Rpg -> 100k,0603
- R23: renamed from R20; value 806k Rfbt -> 806k,0603
- R24: renamed from R21; value 91k Rfbb -> 91k,0603
- renumbered C10 to C11, J7 to J9, U3 to U4, U4 to U5, U5 to U6
Connections:
- net GNDD2 is gone; now on net GNDD: C12.2, C13.2, R24.2, U6.3 (AGND), U6.8 (GND)
- net GNDD: now also Q5.2 (S), R11.1, U3.1 (GND), U3.2 (GND), U3.3 (GND), U3.7 (GND); no longer R19.2
- net VRAW: now also R19.2, Q6.2 (S); no longer C12.1, R22.1, U6.1 (EN), U6.10 (VIN), U6.2 (MODE)
- net at J7.2 (Pin_2): now also R20.1
- net at J7.3 (Pin_3): now also R21.1; no longer R20.1
- net at J7.4 (Pin_4): now also R16.1, R17.2, U5.3 (VIN1), U5.5 (MODE); no longer R21.1
- net at BT1.1 (+), U5.6 (VIN2): now also R12.1, U3.4 (IN), U3.5 (IN), U3.6 (IN)
- net at R19.1: now also Q5.3 (D), Q6.1 (G)
- net at J8.2 (Pin_2): now also J9.B5 (CC2)
- net at J8.3 (Pin_3): now also J9.A5 (CC1); no longer J9.B5 (CC2)
- net at J8.4 (Pin_4): now also J9.A9 (VBUS), J9.B9 (VBUS); no longer J9.A5 (CC1)
- new net: C12.1, Q6.3 (D), R22.1, U6.1 (EN), U6.10 (VIN), U6.2 (MODE)
- new net: Q5.1 (G), R18.2
- new net MOSFET_GATE_SENSOR: R18.1
- new net VCC_BAT: R11.2, R12.2
- no-connect marks 4 -> 0
Other:
- moved on the sheet: BT1, C11, C12, C13, J9, L2, R16, R17, R19, R20, R21, R22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

Commit message: dev
Other:
- note added: "DC-DC BUCK-BOOST converter, VRAW to 5V0 Regulated"
- note removed: "DC-DC BUCK-BOOST converter, VRAW to 5V5 Regulated"
Changed lines of the file:
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@@
 		)
 	)
-	(text "DC-DC BUCK-BOOST converter, VRAW to 5V5 Regulated\n\n"
+	(text "DC-DC BUCK-BOOST converter, VRAW to 5V0 Regulated\n\n"
 		(exclude_from_sim no)
 		(at 152.146 93.726 0)
