File: KiCAD/FlameSensorSender V2/FlameSensorSender.kicad_sch (KiCad schematic)
At the start: 35 parts, among them J1 SWD, J2 SWD, J3 Conn_01x06_Socket, J4 JST-PH PHR-2, J5 Conn_01x01_Socket, J6 Conn_01x01_Socket, Q1 AO3401A, Q2 AO3400A, Q3 AO3401A, Q4 AO3400A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

Commit message: dev
Parts:
- removed Q1, Q3: AO3401A, Package_TO_SOT_SMD:SOT-23-3, symbol Transistor_FET:AO3401A
- removed Q2, Q4: AO3400A, Package_TO_SOT_SMD:SOT-23, symbol Transistor_FET:AO3400A
- removed R2, R7: 47k,0603, Resistor_SMD:R_0603_1608Metric_Pad0.98x0.95mm_HandSolder, symbol Device:R
- removed R3: 10,0603, Resistor_SMD:R_0603_1608Metric_Pad0.98x0.95mm_HandSolder, symbol Device:R
- added C8, C9: 1uF,0603, Capacitor_SMD:C_0603_1608Metric_Pad1.08x0.95mm_HandSolder, symbol Device:C
- added U3, U4: TPS22929D, Package_TO_SOT_SMD:SOT-23-6, symbol Power_Management:TPS22929D
- R5: renamed from R8; value 10,0603 -> 10k,0603
- renumbered C8 to C10, R4 to R2, R5 to R3, R6 to R4, R9 to R6, R10 to R7
Connections:
- net +3V3: now also C8.1, U3.4 (VIN), U3.6 (VIN)
- net +5V0: now also C9.1, U4.4 (VIN), U4.6 (VIN)
- net BUZZER: now also R5.1; no longer R5.2
- net GNDD: now also C8.2, C9.2, U3.2 (GND), U3.5 (GND), U4.2 (GND), U4.5 (GND)
- net LORA_BUSY: now also U1.20 (PB2); no longer U1.13 (PA3)
- net MOSFET_GATE_LORA: now also U3.3 (ON)
- net at FB1.1: now also U3.1 (VOUT)
- net at R7.1: now also U4.1 (VOUT)
- new net: R5.2, U4.3 (ON)
Other:
- moved on the sheet: BZ1, C6, FB1, J4, J5, J6, R5, R7
